File: usb.kicad_sch (KiCad schematic)
At the start: 7 parts, among them J6 USB_C_Receptacle_USB2.0, U5 USBLC6-2P6

Commit message: add ethernet in schematic
Parts:
- removed J6: USB_C_Receptacle_USB2.0, Connector_USB:USB_C_Receptacle_GCT_USB4105-xx-A_16P_TopMnt_Horizontal, symbol Connector:USB_C_Receptacle_USB2.0
- added J8: USB_C_Receptacle_USB2.0_16P, Connector_USB:USB_C_Receptacle_G-Switch_GT-USB-7051x, symbol Connector:USB_C_Receptacle_USB2.0_16P
Connections:
- net GND: now also J8.A1 (GND), J8.A12 (GND), J8.B1 (GND), J8.B12 (GND), J8.S1 (SHIELD)
- net at U5.4 (I/O2): now also J8.A7 (D-), J8.B7 (D-)
- net at D1.2 (A), U5.5 (VBUS): now also J8.A4 (VBUS), J8.A9 (VBUS), J8.B4 (VBUS), J8.B9 (VBUS)
- net at U5.6 (I/O1): now also J8.A6 (D+), J8.B6 (D+)
- net at R11.1: now also J8.A5 (CC1)
- net at R12.1: now also J8.B5 (CC2)
Changed lines of the file:
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@@
+	(wire
+		(pts
+			(xy 135.89 115.57) (xy 135.89 111.76)
+		)
+		(stroke
+			(width 0)
+			(type default)
+		)
+	)
 	(wire
 		(pts
 			(xy 161.29 78.74) (xy 163.83 78.74)
+		)
+		(stroke
+			(width 0)
+			(type default)
+		)
+	)
+	(wire
+		(pts
+			(xy 128.27 115.57) (xy 128.27 111.76)
 		)
 		(stroke
@@
 	)
 	(symbol
-		(lib_id "power:GND")
-		(at 128.27 111.76 0)
+		(lib_id "Connector:USB_C_Receptacle_USB2.0_16P")
+		(at 135.89 88.9 0)
 		(unit 1)
 		(exclude_from_sim no)
@@
 		(dnp no)
 		(fields_autoplaced yes)
+		(property "Reference" "J8"
+			(at 135.89 66.04 0)
+			(effects
+				(font
+					(size 1.27 1.27)
+				)
+			)
+		)
+		(property "Value" "USB_C_Receptacle_USB2.0_16P"
+			(at 135.89 68.58 0)
+			(effects
+				(font
+					(size 1.27 1.27)
+				)
+			)
+		)
+		(property "Footprint" "Connector_USB:USB_C_Receptacle_G-Switch_GT-USB-7051x"
+			(at 139.7 88.9 0)
+			(effects
+				(font
+					(size 1.27 1.27)
+				)
+				(hide yes)
+			)
+		)
+		(property "Datasheet" "https://www.usb.org/sites/default/files/documents/usb_type-c.zip"
+			(at 139.7 88.9 0)
+			(effects
+				(font
+					(size 1.27 1.27)
+				)
+				(hide yes)
+			)
+		)
+		(property "Description" "USB 2.0-only 16P Type-C Receptacle connector"
+			(at 135.89 88.9 0)
+			(effects
+				(font
+					(size 1.27 1.27)
+				)
+				(hide yes)
+			)
+		)
+		(pin "B1"
+		)
+		(pin "A4"
+		)
+		(pin "A8"
+		)
+		(pin "S1"
+		)
+		(pin "A5"
+		)
+		(pin "A7"
+		)
+		(pin "A9"
+		)
+		(pin "B6"
+		)
+		(pin "A12"
+		)
+		(pin "B5"
+		)
+		(pin "A6"
+		)
+		(pin "B8"
+		)
+		(pin "B4"
+		)
+		(pin "A1"
+		)
+		(pin "B9"
+		)
+		(pin "B7"
+		)
+		(pin "B12"
+		)
+		(instances
+			(project "carte_lidar"
+				(path "/8c7c486d-228e-4b66-b6d5-0b7cf34b4d2b/5cfb2dd4-2139-45de-9d20-4a120a5e9868"
+					(reference "J8")
+					(unit 1)
+				)
+			)
+		)
+	)
+	(symbol
+		(lib_id "power:GND")
+		(at 128.27 115.57 0)
+		(unit 1)
+		(exclude_from_sim no)
+		(in_bom yes)
+		(on_board yes)
+		(dnp no)
+		(fields_autoplaced yes)
 		(property "Reference" "#PWR037"
-			(at 128.27 118.11 0)
+			(at 128.27 121.92 0)
 			(effects
 				(font
@@
 		)
 		(property "Value" "GND"
-			(at 128.27 116.84 0)
+			(at 128.27 120.65 0)
 			(effects
 				(font
@@
 		)
 		(property "Footprint" ""
-			(at 128.27 111.76 0)
+			(at 128.27 115.57 0)
 			(effects
 				(font
@@
 		)
 		(property "Datasheet" ""
-			(at 128.27 111.76 0)
+			(at 128.27 115.57 0)
 			(effects
 				(font
@@
 		)
 		(property "Description" ""
-			(at 128.27 111.76 0)
+			(at 128.27 115.57 0)
 			(effects
 				(font
@@
 	)
 	(symbol
-		(lib_id "Connector:USB_C_Receptacle_USB2.0")
-		(at 135.89 88.9 0)
+		(lib_id "power:GND")
+		(at 135.89 115.57 0)
 		(unit 1)
 		(exclude_from_sim no)
@@
 		(dnp no)
 		(fields_autoplaced yes)
-		(property "Reference" "J6"
-			(at 135.89 66.04 0)
-			(effects
-				(font
-					(size 1.27 1.27)
-				)
-			)
-		)
-		(property "Value" "USB_C_Receptacle_USB2.0"
-			(at 135.89 68.58 0)
-			(effects
-				(font
-					(size 1.27 1.27)
-				)
-			)
-		)
-		(property "Footprint" "Connector_USB:USB_C_Receptacle_GCT_USB4105-xx-A_16P_TopMnt_Horizontal"
-			(at 139.7 88.9 0)
-			(effects
-				(font
-					(size 1.27 1.27)
-				)
-				(hide yes)
-			)
-		)
-		(property "Datasheet" "https://www.usb.org/sites/default/files/documents/usb_type-c.zip"
-			(at 139.7 88.9 0)
+		(property "Reference" "#PWR038"
+			(at 135.89 121.92 0)
+			(effects
+				(font
+					(size 1.27 1.27)
+				)
+				(hide yes)
+			)
+		)
+		(property "Value" "GND"
+			(at 135.89 120.65 0)
+			(effects
+				(font
+					(size 1.27 1.27)
+				)
+			)
+		)
+		(property "Footprint" ""
+			(at 135.89 115.57 0)
+			(effects
+				(font
+					(size 1.27 1.27)
+				)
+				(hide yes)
+			)
+		)
+		(property "Datasheet" ""
+			(at 135.89 115.57 0)
 			(effects
 				(font
@@
 		)
 		(property "Description" ""
-			(at 135.89 88.9 0)
-			(effects
-				(font
-					(size 1.27 1.27)
-				)
-				(hide yes)
-			)
-		)
-		(pin "A1"
-		)
-		(pin "A12"
-		)
-		(pin "A4"
-		)
-		(pin "A5"
-		)
-		(pin "A6"
-		)
-		(pin "A7"
-		)
-		(pin "A8"
-		)
-		(pin "A9"
-		)
-		(pin "B1"
-		)
-		(pin "B12"
-		)
-		(pin "B4"
-		)
-		(pin "B5"
-		)
-		(pin "B6"
-		)
-		(pin "B7"
-		)
-		(pin "B8"
-		)
-		(pin "B9"
-		)
-		(pin "S1"
-		)
-		(instances
-			(project "carte_lidar"
-				(path "/8c7c486d-228e-4b66-b6d5-0b7cf34b4d2b/5cfb2dd4-2139-45de-9d20-4a120a5e9868"
-					(reference "J6")
-					(unit 1)
-				)
-			)
-		)
-	)
-	(symbol
-		(lib_id "power:GND")
-		(at 135.89 111.76 0)
-		(unit 1)
-		(exclude_from_sim no)
-		(in_bom yes)
-		(on_board yes)
-		(dnp no)
-		(fields_autoplaced yes)
-		(property "Reference" "#PWR038"
-			(at 135.89 118.11 0)
-			(effects
-				(font
-					(size 1.27 1.27)
-				)
-				(hide yes)
-			)
-		)
-		(property "Value" "GND"
-			(at 135.89 116.84 0)
-			(effects
-				(font
-					(size 1.27 1.27)
-				)
-			)
-		)
-		(property "Footprint" ""
-			(at 135.89 111.76 0)
-			(effects
-				(font
-					(size 1.27 1.27)
-				)
-				(hide yes)
-			)
-		)
-		(property "Datasheet" ""
-			(at 135.89 111.76 0)
-			(effects
-				(font
-					(size 1.27 1.27)
-				)
-				(hide yes)
-			)
-		)
-		(property "Description" ""
-			(at 135.89 111.76 0)
-			(effects
-				(font
+			(at 135.89 115.57 0)
+			(effects
+				(font
