File: ethernet.kicad_sch (KiCad schematic)
At the start: 14 parts, among them J7 RJ45_LED_Shielded, U8 W5500, X2 S2D25.000000B20F30T

Commit message: update all
Parts:
- added J6, J9: Conn_01x06_Socket, Connector_PinHeader_2.54mm:PinHeader_1x06_P2.54mm_Vertical, symbol Connector:Conn_01x06_Socket
Connections:
- net +3V3: now also J9.4 (Pin_4), J9.5 (Pin_5)
- net GND: now also J6.1 (Pin_1), J6.2 (Pin_2), J9.6 (Pin_6)
- net eth_int: now also J6.6 (Pin_6)
- net eth_miso: now also J9.1 (Pin_1)
- net eth_mosi: now also J6.3 (Pin_3)
- net eth_rst: now also J9.2 (Pin_2)
- net eth_sclk: now also J6.4 (Pin_4)
- net eth_scs: now also J6.5 (Pin_5)
Other:
- note added: "remplacé par le shield"
- moved on the sheet: C29, C30, J7, LED3, LED4, LED5, LED6, R19, R20, R21, R22, R23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
