File: power.kicad_sch (KiCad schematic)
At the start: 37 parts, among them J2 Conn_01x02_Pin, U1 TPS54302, U4 TPS54302, U6 NM/AMS1117-3.3

Commit message: update
Parts:
- added F1: JK-SMD300L-24V, Fuse:Fuse_2920_7451Metric, symbol Device:Polyfuse
- added JP1, JP2: SolderJumper_2_Open, Jumper:SolderJumper-2_P1.3mm_Open_RoundedPad1.0x1.5mm, symbol Jumper:SolderJumper_2_Open
- added U9: NM/AMS1117-3.3, Package_TO_SOT_SMD:SOT-223-3_TabPin2, symbol Regulator_Linear:AMS1117-3.3
- R17: value 5.1k -> 10k
Connections:
- net +3V3: now also JP1.2 (B), JP2.2 (B); no longer U6.2 (VO)
- net +5V: now also U9.3 (VI)
- net GND: now also U9.1 (GND)
- net VBAT: now also F1.1; no longer C1.1, C2.1, C3.1, R17.2, U1.3 (VIN)
- new net: JP2.1 (A), U9.2 (VO)
- new net: JP1.1 (A), U6.2 (VO)
- new net VBAT_FUZED: C1.1, C2.1, C3.1, F1.2, R17.2, U1.3 (VIN)
Other:
- moved on the sheet: J2
